File: PCB/PCBGNDPlane.sch (EAGLE design)
At the start: 222 parts, among them Q1 FS8205A, U1 ESP32-S3HOLE, U2 ME6211C33M5G

Commit message: Finished PCB Board and Schematic
Parts:
- added U$100, U$101, U$102, U$103, U$104, U$105, U$97, U$98, U$99: WS2812B5050, Led-WS2812B:WS2812B5050
Connections:
- net N$31 renamed TPPROG
- net N$32 renamed DWCS
- net N$33 renamed DWOC
- net N$34 renamed DWOD
- net N$36 renamed DWVCC
- new net N$100: U$100.LED_DI, U$99.LED_DO
- new net N$101: U$100.LED_DO, U$101.LED_DI
- new net N$102: U$101.LED_DO, U$102.LED_DI
- new net N$103: U$102.LED_DO, U$103.LED_DI
- new net N$104: U$103.LED_DO, U$104.LED_DI
- new net N$105: U$104.LED_DO, U$105.LED_DI
- new net N$106: U$67.LED_DO, U$97.LED_DI
- net GND: now also U$100.LED_GND, U$101.LED_GND, U$102.LED_GND, U$103.LED_GND, U$104.LED_GND, U$105.LED_GND, U$67.LED_GND, U$97.LED_GND, U$98.LED_GND, U$99.LED_GND
- net N$35: now also U$97.LED_DO, U$98.LED_DI; no longer U$67.LED_GND
- net N$79: now also U$98.LED_DO, U$99.LED_DI; no longer U$67.LED_VDD
- net VCC: now also U$100.LED_VDD, U$101.LED_VDD, U$102.LED_VDD, U$103.LED_VDD, U$104.LED_VDD, U$105.LED_VDD, U$67.LED_VDD, U$97.LED_VDD, U$98.LED_VDD, U$99.LED_VDD
