File: PCB/ModernWoodPCB.brd (EAGLE design)
At the start: 428.5 x 125 mm, 231 parts, among them Q1 FS8205A, U1 ESP32-S3HOLE, U2 ME6211C33M5G

Commit message: Revision 2 of PCB and Finished
Parts:
- removed Q1: FS8205A, FS8205A:SOP65P640X120-8N
- added Q2: FS8205, FS8205:SOT95P280X145-6N
Connections:
- removed net DWOC: Q1.5, U$96.3
- removed net DWOD: Q1.4, U$96.1
- new net N$31: Q2.6, U$96.1
- new net N$32: Q2.4, U$96.3
- net B-: now also Q2.1; no longer Q1.2, Q1.3
- net GND: now also Q2.3; no longer Q1.6, Q1.7
Routing:
- net DWOC: track 18.1 -> 0.00 mm, vias 2 -> 0
- net N$31: track 0.00 -> 16.0 mm
- net DWOD: track 9.83 -> 0.00 mm
- net N$32: track 0.00 -> 9.79 mm
- net B-: track 45.3 -> 51.7 mm
- net GND: track 679.5 -> 676.7 mm
Other:
- board text added: "JLCJLCJLCJLC"
